File: pcb/WiFi_Frauder_DEV/WiFi_Frauder_DEV.kicad_pcb (KiCad board)
At the start: 2 copper layers, 93.4 x 64.5 mm, 9 parts, among them SW1 BTN_DOWN, SW2 BTN_UP, SW3 BTN_ENTER, U1 ESP32-DevKitC, U2 DM-OLED096-636

Commit message: feat: revision PCB from 0 to 1
Parts:
- added REF**: OSHW-Logo_5.7x6mm_SilkScreen, Symbol:OSHW-Logo_5.7x6mm_SilkScreen, F.Cu at (178.3, 116.4)
- added REF**: KiCad-Logo2_5mm_SilkScreen, Symbol:KiCad-Logo2_5mm_SilkScreen, F.Cu at (165.8, 116.5)
Connections:
- net Net-(U1-GPIO21) renamed /BTN_ENTER_NET
- net Net-(U1-GPIO22) renamed /BTN_UP_NET
- net Net-(U1-GPIO23) renamed /BTN_DOWN_NET
- net SCL renamed /OLED_SCL_NET
- net SDA renamed /OLED_SDA_NET
Routing:
- net GND: track 209.1 -> 217.1 mm
- net /BTN_ENTER_NET: track 80.1 -> 82.0 mm
- net +5V: track 231.6 -> 233.2 mm
- added copper zone on B.Cu, net GND
- added copper zone on F.Cu, net GND
Other:
- board text added: "WiFi Frauder REV 1"
- board text removed: "WiFi Frauder REV 0"

Commit message: feat: revistion pcb to rev2
Parts:
- removed REF**: OSHW-Logo_5.7x6mm_SilkScreen, Symbol:OSHW-Logo_5.7x6mm_SilkScreen
- removed REF**: KiCad-Logo2_5mm_SilkScreen, Symbol:KiCad-Logo2_5mm_SilkScreen
- R1, R2, R3: footprint Capacitor_SMD:C_0805_2012Metric -> Resistor_THT:R_Axial_DIN0207_L6.3mm_D2.5mm_P10.16mm_Horizontal
- moved G*** 56.9 mm to (133.0, 121.6)
- moved U1 36.7 mm to (128.0, 77.1)
- moved R1 31.2 mm to (165.7, 106.7), turned to 0 degrees
- moved SW1 28.7 mm to (152.8, 105.0)
- moved R3 20.5 mm to (165.7, 122.5), turned to 0 degrees
- moved SW3 19.8 mm to (152.8, 120.2)
- moved U2 19.3 mm to (133.1, 100.2)
- moved SW2 17.2 mm to (152.8, 88.8)
- moved R2 16.4 mm to (165.7, 90.8), turned to 0 degrees
Routing:
- net GND: track 217.1 -> 38.8 mm, vias 1 -> 7
- net +5V: track 233.2 -> 125.6 mm, vias 1 -> 0
- net /BTN_ENTER_NET: track 82.0 -> 165.5 mm, vias 1 -> 0
- net /BTN_UP_NET: track 48.8 -> 117.1 mm
- net /BTN_DOWN_NET: track 65.0 -> 121.1 mm
- net /OLED_SDA_NET: track 66.0 -> 93.3 mm
- net /OLED_SCL_NET: track 72.2 -> 79.6 mm
Other:
- board size 93.4 x 64.5 mm -> 67.5 x 95.6 mm
- board text added: "Firmware and Hardware by"
- board text added: "REV 2"
- board text added: "WiFi Frauder"
- board text added: "un4ckn0wl3z"
- board text removed: "By un4ckn0wl3z"
- board text removed: "WiFi Frauder REV 1"
- board text removed: "eavesdropper.dev"

Commit message: feat: re-design pcb
Connections:
- U1 pad 20: /OLED_SCL_NET -> unconnected-(U1-SD_CLK/GPIO6-Pad20)
- U1 pad 21: /OLED_SDA_NET -> unconnected-(U1-SD_DATA0/GPIO7-Pad21)
- U1 pad 27: unconnected-(U1-GPIO16-Pad27) -> /OLED_SDA_NET
- U1 pad 28: unconnected-(U1-GPIO17-Pad28) -> /OLED_SCL_NET
Routing:
- net /OLED_SCL_NET: track 79.6 -> 104.9 mm
- net /OLED_SDA_NET: track 93.3 -> 77.9 mm
- net /BTN_ENTER_NET: track 165.5 -> 164.1 mm
Other:
- board text added: "REV 3"
- board text removed: "REV 2"
Changed lines of the file:
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@@
 	(title_block
 		(title "WiFi_Frauder_DEV ")
-		(date "2025-06-12")
-		(rev "2")
+		(date "2025-06-14")
+		(rev "3")
 		(company "By Anuwat Khongchuai (un4ckn0wl3z)")
 	)
@@
 	(net 9 "unconnected-(U1-MTCK{slash}GPIO13{slash}ADC2_CH4-Pad15)")
 	(net 10 "unconnected-(U1-SENSOR_VN{slash}GPIO39{slash}ADC1_CH3-Pad4)")
-	(net 11 "unconnected-(U1-GPIO16-Pad27)")
+	(net 11 "unconnected-(U1-SD_DATA0{slash}GPIO7-Pad21)")
 	(net 12 "unconnected-(U1-MTDO{slash}GPIO15{slash}ADC2_CH3-Pad23)")
 	(net 13 "unconnected-(U1-VDET_2{slash}GPIO35{slash}ADC1_CH7-Pad6)")
@@
 	(net 28 "unconnected-(U1-ADC2_CH7{slash}GPIO27-Pad11)")
 	(net 29 "unconnected-(U1-3V3-Pad1)")
-	(net 30 "unconnected-(U1-GPIO17-Pad28)")
+	(net 30 "unconnected-(U1-SD_CLK{slash}GPIO6-Pad20)")
 	(net 31 "unconnected-(U1-SD_DATA2{slash}GPIO9-Pad16)")
 	(net 32 "unconnected-(U1-GPIO19-Pad31)")
@@
 			(layers "*.Cu" "*.Mask")
 			(remove_unused_layers no)
-			(net 33 "/OLED_SCL_NET")
+			(net 30 "unconnected-(U1-SD_CLK{slash}GPIO6-Pad20)")
 			(pinfunction "SD_CLK/GPIO6")
-			(pintype "bidirectional")
+			(pintype "bidirectional+no_connect")
 		)
 		(pad "21" thru_hole oval
@@
 			(layers "*.Cu" "*.Mask")
 			(remove_unused_layers no)
-			(net 23 "/OLED_SDA_NET")
+			(net 11 "unconnected-(U1-SD_DATA0{slash}GPIO7-Pad21)")
 			(pinfunction "SD_DATA0/GPIO7")
-			(pintype "bidirectional")
+			(pintype "bidirectional+no_connect")
 		)
 		(pad "22" thru_hole oval
@@
 			(layers "*.Cu" "*.Mask")
 			(remove_unused_layers no)
-			(net 11 "unconnected-(U1-GPIO16-Pad27)")
+			(net 23 "/OLED_SDA_NET")
 			(pinfunction "GPIO16")
-			(pintype "bidirectional+no_connect")
+			(pintype "bidirectional")
 		)
 		(pad "28" thru_hole oval
@@
 			(layers "*.Cu" "*.Mask")
 			(remove_unused_layers no)
-			(net 30 "unconnected-(U1-GPIO17-Pad28)")
+			(net 33 "/OLED_SCL_NET")
 			(pinfunction "GPIO17")
-			(pintype "bidirectional+no_connect")
+			(pintype "bidirectional")
 		)
 		(pad "29" thru_hole oval
@@
 		)
 	)
-	(gr_text "REV 2"
+	(gr_text "REV 3"
 		(at 149.40875 131.9 0)
 		(layer "F.SilkS")
@@
 	)
 	(segment
-		(start 133.20531 44.2)
+		(start 134.90531 45.9)
 		(end 140.70531 51.7)
 		(width 0.2)
@@
 	)
 	(segment
-		(start 116.40875 102.965501)
-		(end 116.40875 47.8)
+		(start 152.75875 120.15)
+		(end 133.593249 120.15)
 		(width 0.2)
 		(layer "B.Cu")
@@
 	)
 	(segment
-		(start 152.75875 120.15)
-		(end 133.593249 120.15)
+		(start 133.593249 120.15)
+		(end 116.40875 102.965501)
 		(width 0.2)
 		(layer "B.Cu")
@@
 	)
 	(segment
-		(start 116.40875 47.8)
-		(end 120.00875 44.2)
+		(start 118.30875 45.9)
+		(end 134.90531 45.9)
 		(width 0.2)
 		(layer "B.Cu")
@@
 	)
 	(segment
-		(start 120.00875 44.2)
-		(end 133.20531 44.2)
+		(start 116.40875 102.965501)
+		(end 116.40875 47.8)
 		(width 0.2)
 		(layer "B.Cu")
@@
 	)
 	(segment
-		(start 133.593249 120.15)
-		(end 116.40875 102.965501)
+		(start 116.40875 47.8)
+		(end 118.30875 45.9)
 		(width 0.2)
 		(layer "B.Cu")
@@
 	)
 	(segment
-		(start 124.80875 65.1)
-		(end 124.80875 83.9)
+		(start 126.30875 90.3)
+		(end 128.10875 92.1)
+		(width 0.2)
+		(layer "B.Cu")
+		(net 23)
+	)
+	(segment
+		(start 128.40875 61.5)
+		(end 149.3 61.5)
 		(width 0.2)
 		(layer "B.Cu")
@@
 	)
 	(segment
-		(start 128.10875 92.1)
-		(end 134.80875 92.1)
+		(start 149.309554 61.509554)
+		(end 155.94531 54.873798)
 		(width 0.2)
 		(layer "B.Cu")
@@
 	)
 	(segment
-		(start 171.18259 55.12616)
-		(end 164.80875 61.5)
+		(start 126.30875 85.4)
+		(end 126.30875 90.3)
 		(width 0.2)
 		(layer "B.Cu")
@@
 	)
 	(segment
-		(start 124.80875 83.9)
-		(end 126.30875 85.4)
+		(start 134.80875 92.1)
+		(end 136.91875 89.99)
 		(width 0.2)
 		(layer "B.Cu")
@@
 	)
 	(segment
-		(start 136.91875 89.99)
-		(end 136.91875 88.7125)
+		(start 155.94531 54.873798)
+		(end 155.94531 51.7)
 		(width 0.2)
 		(layer "B.Cu")
@@
 	)
 	(segment
-		(start 171.18259 51.70368)
-		(end 171.18259 55.12616)
+		(start 149.3 61.5)
+		(end 149.309554 61.509554)
 		(width 0.2)
 		(layer "B.Cu")
@@
 	)
 	(segment
-		(start 126.30875 85.4)
-		(end 126.30875 90.3)
+		(start 136.91875 89.99)
+		(end 136.91875 88.7125)
 		(width 0.2)
 		(layer "B.Cu")
@@
 	)
 	(segment
-		(start 164.80875 61.5)
-		(end 128.40875 61.5)
+		(start 124.80875 65.1)
+		(end 124.80875 83.9)
 		(width 0.2)
 		(layer "B.Cu")
@@
 	)
 	(segment
-		(start 134.80875 92.1)
-		(end 136.91875 89.99)
+		(start 124.80875 83.9)
+		(end 126.30875 85.4)
 		(width 0.2)
 		(layer "B.Cu")
@@
 	)
 	(segment
-		(start 126.30875 90.3)
-		(end 128.10875 92.1)
+		(start 128.10875 92.1)
+		(end 134.80875 92.1)
 		(width 0.2)
 		(layer "B.Cu")
@@
 	)
 	(segment
-		(start 177.50875 52.3)
-		(end 176.91243 51.70368)
+		(start 153.40531 50.89469)
+		(end 153.40531 51.7)
 		(width 0.2)
 		(layer "B.Cu")
@@
 	)
 	(segment
-		(start 177.50875 79.5)
-		(end 177.50875 52.3)
+		(start 137.69125 85.4)
+		(end 162.90875 85.4)
 		(width 0.2)
 		(layer "B.Cu")
@@
 	)
 	(segment
-		(start 176.91243 51.70368)
-		(end 173.72259 51.70368)
+		(start 134.37875 88.7125)
+		(end 137.69125 85.4)
 		(width 0.2)
 		(layer "B.Cu")
@@
 	)
 	(segment
-		(start 137.69125 85.4)
-		(end 162.90875 85.4)
+		(start 173.1 46.9)
+		(end 157.4 46.9)
 		(width 0.2)
 		(layer "B.Cu")
@@
 	)
 	(segment
-		(start 134.37875 88.7125)
-		(end 137.69125 85.4)
+		(start 177.50875 51.30875)
+		(end 173.1 46.9)
 		(width 0.2)
 		(layer "B.Cu")
@@
 	)
 	(segment
+		(start 157.4 46.9)
+		(end 153.40531 50.89469)
+		(width 0.2)
+		(layer "B.Cu")
+		(net 33)
+	)
+	(segment
 		(start 169.90875 87.1)
 		(end 177.50875 79.5)
@@
 		(net 33)
 	)
+	(segment
+		(start 177.50875 79.5)
+		(end 177.50875 51.30875)
+		(width 0.2)
+		(layer "B.Cu")
+		(net 33)
+	)
 	(zone
 		(net 1)
@@
 		(polygon
 			(pts
-				(xy 114.20875 42) (xy 184.00875 41.7) (xy 183.50875 139.1) (xy 113.80875 139.2)
+				(xy 114 41) (xy 184.2 41) (xy 184 140) (xy 112 140)
 			)
 		)

Commit message: feat: re-designed pcb included extended female socket for GPIO
Parts:
- added J1: Conn_01x19_Socket, Connector_PinSocket_2.54mm:PinSocket_1x19_P2.54mm_Vertical, F.Cu at (128.3, 86.4)
- added J2: Conn_01x19_Socket, Connector_PinSocket_2.54mm:PinSocket_1x19_P2.54mm_Vertical, F.Cu at (174.0, 41.9)
- moved U2 9.02 mm to (134.1, 109.2)
- moved G*** 9.02 mm to (133.9, 130.6)
- moved R1 9.02 mm to (166.7, 115.6)
- moved R2 9.02 mm to (166.7, 99.8)
- moved R3 9.02 mm to (166.7, 131.5)
- moved SW1 9.02 mm to (153.7, 113.9)
- moved SW2 9.02 mm to (153.7, 97.8)
- moved SW3 9.02 mm to (153.7, 129.1)
Connections:
- net +5V renamed 5V
- U1 pad 1: unconnected-(U1-3V3-Pad1) -> 3V3
- U1 pad 10: unconnected-(U1-DAC_2/ADC2_CH9/GPIO26-Pad10) -> /GPIO26
- U1 pad 11: unconnected-(U1-ADC2_CH7/GPIO27-Pad11) -> /GPIO27
- U1 pad 12: unconnected-(U1-MTMS/GPIO14/ADC2_CH6-Pad12) -> /GPIO14
- U1 pad 13: unconnected-(U1-MTDI/GPIO12/ADC2_CH5-Pad13) -> /GPIO12
- U1 pad 15: unconnected-(U1-MTCK/GPIO13/ADC2_CH4-Pad15) -> /GPIO13
- U1 pad 16: unconnected-(U1-SD_DATA2/GPIO9-Pad16) -> /GPIO9
- U1 pad 17: unconnected-(U1-SD_DATA3/GPIO10-Pad17) -> /GPIO10
- U1 pad 18: unconnected-(U1-CMD-Pad18) -> /CMD
- U1 pad 2: unconnected-(U1-CHIP_PU-Pad2) -> /CHIP_PU
- U1 pad 20: unconnected-(U1-SD_CLK/GPIO6-Pad20) -> /GPIO6
- U1 pad 21: unconnected-(U1-SD_DATA0/GPIO7-Pad21) -> /GPIO7
- U1 pad 22: unconnected-(U1-SD_DATA1/GPIO8-Pad22) -> /GPIO8
- U1 pad 23: unconnected-(U1-MTDO/GPIO15/ADC2_CH3-Pad23) -> /GPIO15
- U1 pad 24: unconnected-(U1-ADC2_CH2/GPIO2-Pad24) -> /GPIO2
- U1 pad 25: unconnected-(U1-GPIO0/BOOT/ADC2_CH1-Pad25) -> /GPIO0
- U1 pad 26: unconnected-(U1-ADC2_CH0/GPIO4-Pad26) -> /GPIO4
- U1 pad 29: unconnected-(U1-GPIO5-Pad29) -> /GPIO5
- U1 pad 3: unconnected-(U1-SENSOR_VP/GPIO36/ADC1_CH0-Pad3) -> /GPIO36
- U1 pad 30: unconnected-(U1-GPIO18-Pad30) -> /GPIO18
- U1 pad 31: unconnected-(U1-GPIO19-Pad31) -> /GPIO19
- U1 pad 34: unconnected-(U1-U0RXD/GPIO3-Pad34) -> /GPIO3
- U1 pad 35: unconnected-(U1-U0TXD/GPIO1-Pad35) -> /GPIO1
- U1 pad 4: unconnected-(U1-SENSOR_VN/GPIO39/ADC1_CH3-Pad4) -> /GPIO39
- U1 pad 5: unconnected-(U1-VDET_1/GPIO34/ADC1_CH6-Pad5) -> /GPIO34
- U1 pad 6: unconnected-(U1-VDET_2/GPIO35/ADC1_CH7-Pad6) -> /GPIO35
- U1 pad 7: unconnected-(U1-32K_XP/GPIO32/ADC1_CH4-Pad7) -> /GPIO32
- U1 pad 8: unconnected-(U1-32K_XN/GPIO33/ADC1_CH5-Pad8) -> /GPIO33
- U1 pad 9: unconnected-(U1-DAC_1/ADC2_CH8/GPIO25-Pad9) -> /GPIO25
Routing:
- net 5V: track 125.6 -> 149.8 mm
- net /OLED_SDA_NET: track 77.9 -> 99.4 mm
- net /BTN_DOWN_NET: track 121.1 -> 141.4 mm
- net /BTN_UP_NET: track 117.1 -> 137.1 mm
- net /OLED_SCL_NET: track 104.9 -> 123.9 mm
- net /BTN_ENTER_NET: track 164.1 -> 182.7 mm
- net GND: track 38.8 -> 53.2 mm, vias 7 -> 10
- net /GPIO6: track 0.00 -> 11.4 mm
- net /GPIO25: track 0.00 -> 11.4 mm
- net /GPIO39: track 0.00 -> 11.4 mm
- net /GPIO14: track 0.00 -> 11.4 mm
- net /GPIO34: track 0.00 -> 11.3 mm
- net /GPIO33: track 0.00 -> 11.2 mm
- net /GPIO12: track 0.00 -> 11.2 mm
- net /GPIO32: track 0.00 -> 11.2 mm
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Other:
- board size 67.5 x 95.6 mm -> 67.5 x 113.4 mm
